File: Flyback Designs/Flyback_PCBs/r10 Atverter_Fly/Atverter_Fly.kicad_pcb (KiCad board)
At the start: 2 copper layers, 118 x 68.8 mm, 64 parts, among them T1 Transformer_1P_1S, U1 PVI5080NPBF

Commit message: Add files via upload
Parts:
- Vin(+) GND: renamed from GND_Vin(+)1
- Vout(+) GND: renamed from Vout(+)_GND1
- moved Cosc1 0.49 mm to (133.5, 80.4)
- renumbered ATmega1 to ATmega, CDTR1 to CDTR, CSup1 to CSup, Copto1 to Copto, Cout1 to Cout, GateDriver1 to GateDriver, MOSFET1 to MOSFET, PowGNDs1 to PowGNDs, RDTR1 to RDTR, RPi1 to RPi, SignGNDs1 to SignGNDs, I_InHeader1 to Vin_InHeader, Xtal1 to Xtal
Connections:
- T1 pad 1: Net-(T1-AA) -> unconnected-(ATmega1-AREF-Pad21)
- T1 pad 10: (no net) -> unconnected-(ATmega1-PB0-Pad14)
- T1 pad 11: (no net) -> unconnected-(ATmega1-PB0-Pad14)
- T1 pad 12: (no net) -> unconnected-(ATmega1-PB0-Pad14)
- T1 pad 13: (no net) -> unconnected-(ATmega1-PC4-Pad27)
- T1 pad 14: (no net) -> unconnected-(ATmega1-PC4-Pad27)
- T1 pad 15: (no net) -> unconnected-(ATmega1-PC4-Pad27)
- T1 pad 16: (no net) -> unconnected-(ATmega1-PC4-Pad27)
- T1 pad 2: Net-(D1-A) -> unconnected-(ATmega1-AREF-Pad21)
- T1 pad 3: PGND -> unconnected-(ATmega1-AREF-Pad21)
- T1 pad 4: Net-(T1-SB) -> unconnected-(ATmega1-AREF-Pad21)
- T1 pad 5: (no net) -> unconnected-(ATmega1-AREF-Pad21)
- T1 pad 6: (no net) -> unconnected-(ATmega1-AREF-Pad21)
- T1 pad 7: (no net) -> unconnected-(ATmega1-PB0-Pad14)
- T1 pad 8: (no net) -> unconnected-(ATmega1-PB0-Pad14)
- T1 pad 9: (no net) -> unconnected-(ATmega1-PB0-Pad14)
Routing:
- net AGND: track 53.0 -> 54.4 mm
- net Net-(T1-AA): track 59.7 -> 58.7 mm
- net /+10Vcc: track 92.1 -> 91.5 mm
- net PGND: vias 38 -> 46
- net Net-(D1-A): vias 1 -> 0
- net /Vout(+): vias 18 -> 15
- net /Vin(+): vias 19 -> 14
- added copper zone on F.Cu, net Net-(T1-AA)
